Commit message: Second Commit

File: Universal_Robots_ROS2_Description-humble/urdf/inc/ur_transmissions.xacro (robot description, xacro)
@@ -62,5 +62,5 @@
     </transmission>
     <!-- Trasmission for fake hand -->
-    <!-- <transmission name="${prefix}flange-tool0_trans">
+    <transmission name="${prefix}flange-tool0_trans">
       <type>transmission_interface/SimpleTransmission</type>
       <joint name="${prefix}flange-tool0">
@@ -70,5 +70,5 @@
         <mechanicalReduction>1</mechanicalReduction>
       </actuator>
-    </transmission> -->
+    </transmission>
   </xacro:macro>
 </robot>

File: Universal_Robots_ROS2_Description-humble/urdf/ur.ros2_control.xacro (robot description, xacro)
@@ -127,5 +127,5 @@
       <!-- Per permettere il controllo della fake hand -->
       <!-- NON DIMENTICARTI DI LANCIARLO DA LAUNCH FILE -->
-      <!-- <joint name="${tf_prefix}flange-tool0">
+      <joint name="${tf_prefix}flange-tool0">
           <command_interface name="position"/>
           <command_interface name="velocity"/>
@@ -135,5 +135,5 @@
           <state_interface name="velocity"/>
           <state_interface name="effort"/>
-      </joint> -->
+      </joint>
       <xacro:unless value="${sim_gazebo or sim_ignition}">
         <sensor name="${tf_prefix}tcp_fts_sensor">

File: Universal_Robots_ROS2_Description-humble/urdf/ur.urdf.xacro (robot description, xacro)
@@ -3,12 +3,6 @@
    <!-- robot name parameter -->
    <xacro:arg name="name" default="ur"/>
-   <xacro:arg name="gripper" default="true"/>
    <!-- import main macro -->
-   <xacro:if value="$(arg gripper)">
-      <xacro:include filename="$(find ur_description)/urdf/ur_macro_w_gripper.xacro"/>
-   </xacro:if>
-   <xacro:unless value="$(arg gripper)">
-      <xacro:include filename="$(find ur_description)/urdf/ur_macro.xacro"/>
-   </xacro:unless>
+   <xacro:include filename="$(find ur_description)/urdf/ur_macro.xacro"/>
    <!-- possible 'ur_type' values: ur3, ur3e, ur5, ur5e, ur7e, ur10, ur10e, ur12e, ur16e, ur15, ur20, ur30 -->
    <!-- the default value should raise an error in case this was called without defining the type -->

File: Universal_Robots_ROS2_Description-humble/urdf/ur_macro.xacro (robot description, xacro)
@@ -434,14 +434,7 @@
       <parent link="${tf_prefix}wrist_3_link" />
       <child link="${tf_prefix}flange" />
-      <origin xyz="0 0 0" rpy="0 ${-pi/2.0} ${-pi/2.0}" />
-    </joint>
-    <!-- ROS-Industrial 'tool0' frame - all-zeros tool frame -->
-    <!-- <link name="${tf_prefix}tool0"/>
-    <joint name="${tf_prefix}flange-tool0" type="fixed">
-      <origin xyz="0 0 0" rpy="${pi/2.0} 0 ${pi/2.0}"/>
-      <parent link="${tf_prefix}flange"/>
-      <child link="${tf_prefix}tool0"/>
-    </joint> -->
-    <!-- FAKE TOOL0 LINK (VISIBLE GREEN CUBE) -->
+      <origin xyz="0 0 0.00" rpy="0 ${-pi/2.0} ${-pi/2.0}" />
+    </joint>
+    <!-- FAKE TOOL0 LINK (It Represents a Fake Attached End-Effector) -->
     <link name="${tf_prefix}tool0">
       <visual>
@@ -454,22 +447,16 @@
         </material>
       </visual>
-      <collision>
-        <origin xyz="0 0 0.0" rpy="0 0 0"/>
-        <geometry>
-          <box size="0.02 0.02 0.02"/>
-        </geometry>
-      </collision>
-      <inertial>
-        <mass value="0.01"/>
+     <inertial>
+        <mass value="1e-6"/>
         <origin xyz="0 0 0.0" rpy="0 0 0"/>
         <inertia ixx="1e-5" ixy="0" ixz="0" iyy="1e-5" iyz="0" izz="1e-5"/>
       </inertial>
     </link>
-    <!-- FIXED JOINT FROM wrist_3_link TO tool0 -->
+    <!-- REVOLUTE FAKE JOINT from flange TO tool0 (Cannot be Fixed beacuse it needs to be 'controlled' by MoveIt) -->
     <joint name="${tf_prefix}flange-tool0" type="revolute">
       <parent link="${tf_prefix}wrist_3_link"/>
       <child link="${tf_prefix}tool0"/>
-      <origin xyz="0 0 0" rpy="0 0 0"/>
-      <limit lower="-0.0001" upper="0.0001"
+      <origin xyz="0 0 0.07" rpy="0 0 0"/>
+      <limit lower="-0.00000000000000001" upper="0.0000000000000000001"
              effort="0.001" velocity="0.001"/>
     </joint>
